File: kicad/thorn_matrix.kicad_sch (KiCad schematic)
At the start: 21 parts

Commit message: chore: cleaned up schematic
Parts:
- added SW1: RotaryEncoder, Rotary_Encoder:RotaryEncoder_Alps_EC12E_Vertical_H20mm, symbol Device:RotaryEncoder
- MX1, MX10, MX2, MX3, MX4, MX5, MX6, MX7, MX8, MX9: footprint MX_Only:MXOnly-1U -> MX_Only:MXOnly-1U-NoLED
Connections:
- net GND: now also SW1.C
- net at MX4.2: now also D4.2 (A)
- new net EC1: SW1.A
- new net EC2: SW1.B
Changed lines of the file:
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@@
-	(wire
-		(pts
-			(xy 71.12 49.53) (xy 71.12 50.8)
-		)
-		(stroke
-			(width 0)
-			(type default)
-		)
-	)
 	(wire
 		(pts
@@
 	(wire
 		(pts
+			(xy 71.12 49.3625) (xy 71.12 50.8)
+		)
+		(stroke
+			(width 0)
+			(type default)
+		)
+	)
+	(wire
+		(pts
 			(xy 39.37 78.74) (xy 39.37 92.71)
+		)
+		(stroke
+			(width 0)
+			(type default)
+		)
+	)
+	(wire
+		(pts
+			(xy 133.35 80.01) (xy 140.97 80.01)
 		)
 		(stroke
@@
 		)
 	)
+	(global_label "EC2"
+		(shape input)
+		(at 140.97 82.55 180)
+		(fields_autoplaced yes)
+		(effects
+			(font
+				(size 1.27 1.27)
+			)
+			(justify right)
+		)
+		(property "Intersheetrefs" "${INTERSHEET_REFS}"
+			(at 134.3563 82.55 0)
+			(hide yes)
+			(show_name no)
+			(do_not_autoplace no)
+			(effects
+				(font
+					(size 1.27 1.27)
+				)
+				(justify right)
+			)
+		)
+	)
 	(global_label "COL1"
 		(shape input)
@@
 				)
 				(justify left)
+			)
+		)
+	)
+	(global_label "EC1"
+		(shape input)
+		(at 140.97 77.47 180)
+		(fields_autoplaced yes)
+		(effects
+			(font
+				(size 1.27 1.27)
+			)
+			(justify right)
+		)
+		(property "Intersheetrefs" "${INTERSHEET_REFS}"
+			(at 134.3563 77.47 0)
+			(hide yes)
+			(show_name no)
+			(do_not_autoplace no)
+			(effects
+				(font
+					(size 1.27 1.27)
+				)
+				(justify right)
 			)
 		)
@@
 			)
 		)
-		(property "Footprint" "MX_Only:MXOnly-1U"
+		(property "Footprint" "MX_Only:MXOnly-1U-NoLED"
 			(at 44.45 30.48 0)
 			(hide yes)
@@
 			)
 		)
-		(property "Footprint" "MX_Only:MXOnly-1U"
+		(property "Footprint" "MX_Only:MXOnly-1U-NoLED"
 			(at 66.04 44.2825 0)
 			(hide yes)
@@
 			)
 		)
-		(property "Footprint" "MX_Only:MXOnly-1U"
+		(property "Footprint" "MX_Only:MXOnly-1U-NoLED"
 			(at 44.45 87.63 0)
 			(hide yes)
@@
 			)
 		)
-		(property "Footprint" "MX_Only:MXOnly-1U"
+		(property "Footprint" "MX_Only:MXOnly-1U-NoLED"
 			(at 44.45 73.66 0)
 			(hide yes)
@@
 			)
 		)
-		(property "Footprint" "MX_Only:MXOnly-1U"
+		(property "Footprint" "MX_Only:MXOnly-1U-NoLED"
 			(at 66.04 87.63 0)
 			(hide yes)
@@
 			)
 		)
-		(property "Footprint" "MX_Only:MXOnly-1U"
+		(property "Footprint" "MX_Only:MXOnly-1U-NoLED"
 			(at 66.04 73.66 0)
 			(hide yes)
@@
 			)
 		)
-		(property "Footprint" "MX_Only:MXOnly-1U"
+		(property "Footprint" "MX_Only:MXOnly-1U-NoLED"
 			(at 66.04 30.48 0)
 			(hide yes)
@@
 			)
 		)
-		(property "Footprint" "MX_Only:MXOnly-1U"
+		(property "Footprint" "MX_Only:MXOnly-1U-NoLED"
 			(at 44.45 59.69 0)
 			(hide yes)
@@
 				(path "/08f3c77b-db3c-46f4-9250-f5ee3e1cee68/0f81ac1e-de1d-44ff-8e5e-614f84f00e15"
 					(reference "MX5")
+					(unit 1)
+				)
+			)
+		)
+	)
+	(symbol
+		(lib_id "power:GND")
+		(at 133.35 80.01 270)
+		(unit 1)
+		(body_style 1)
+		(exclude_from_sim no)
+		(in_bom yes)
+		(on_board yes)
+		(in_pos_files yes)
+		(dnp no)
+		(fields_autoplaced yes)
+		(property "Reference" "#PWR025"
+			(at 127 80.01 0)
+			(hide yes)
+			(show_name no)
+			(do_not_autoplace no)
+			(effects
+				(font
+					(size 1.27 1.27)
+				)
+			)
+		)
+		(property "Value" "GND"
+			(at 129.54 80.0099 90)
+			(show_name no)
+			(do_not_autoplace no)
+			(effects
+				(font
+					(size 1.27 1.27)
+				)
+				(justify right)
+			)
+		)
+		(property "Footprint" ""
+			(at 133.35 80.01 0)
+			(hide yes)
+			(show_name no)
+			(do_not_autoplace no)
+			(effects
+				(font
+					(size 1.27 1.27)
+				)
+			)
+		)
+		(property "Datasheet" ""
+			(at 133.35 80.01 0)
+			(hide yes)
+			(show_name no)
+			(do_not_autoplace no)
+			(effects
+				(font
+					(size 1.27 1.27)
+				)
+			)
+		)
+		(property "Description" "Power symbol creates a global label with name \"GND\" , ground"
+			(at 133.35 80.01 0)
+			(hide yes)
+			(show_name no)
+			(do_not_autoplace no)
+			(effects
+				(font
+					(size 1.27 1.27)
+				)
+			)
+		)
+		(pin "1"
+		)
+		(instances
+			(project "thorn"
+				(path "/08f3c77b-db3c-46f4-9250-f5ee3e1cee68/0f81ac1e-de1d-44ff-8e5e-614f84f00e15"
+					(reference "#PWR025")
 					(unit 1)
 				)
@@
 			)
 		)
-		(property "Footprint" "MX_Only:MXOnly-1U"
+		(property "Footprint" "MX_Only:MXOnly-1U-NoLED"
 			(at 66.04 59.69 0)
 			(hide yes)
@@
 	)
 	(symbol
+		(lib_id "Device:RotaryEncoder")
+		(at 148.59 80.01 0)
+		(unit 1)
+		(body_style 1)
+		(exclude_from_sim no)
+		(in_bom yes)
+		(on_board yes)
+		(in_pos_files yes)
+		(dnp no)
+		(fields_autoplaced yes)
+		(property "Reference" "SW1"
+			(at 154.94 78.7399 0)
+			(show_name no)
+			(do_not_autoplace no)
+			(effects
+				(font
+					(size 1.27 1.27)
+				)
+				(justify left)
+			)
+		)
+		(property "Value" "RotaryEncoder"
+			(at 154.94 81.2799 0)
+			(show_name no)
+			(do_not_autoplace no)
+			(effects
+				(font
+					(size 1.27 1.27)
+				)
+				(justify left)
+			)
+		)
+		(property "Footprint" "Rotary_Encoder:RotaryEncoder_Alps_EC12E_Vertical_H20mm"
+			(at 144.78 75.946 0)
+			(hide yes)
+			(show_name no)
+			(do_not_autoplace no)
+			(effects
+				(font
+					(size 1.27 1.27)
+				)
+			)
+		)
+		(property "Datasheet" ""
+			(at 148.59 73.406 0)
+			(hide yes)
+			(show_name no)
+			(do_not_autoplace no)
+			(effects
+				(font
+					(size 1.27 1.27)
+				)
+			)
+		)
+		(property "Description" "Rotary encoder, dual channel, incremental quadrate outputs"
+			(at 148.59 80.01 0)
+			(hide yes)
+			(show_name no)
+			(do_not_autoplace no)
+			(effects
+				(font
+					(size 1.27 1.27)
+				)
+			)
+		)
+		(pin "B"
+		)
+		(pin "C"
+		)
+		(pin "A"
+		)
+		(instances
+			(project "thorn"
+				(path "/08f3c77b-db3c-46f4-9250-f5ee3e1cee68/0f81ac1e-de1d-44ff-8e5e-614f84f00e15"
+					(reference "SW1")
+					(unit 1)
+				)
+			)
+		)
+	)
+	(symbol
 		(lib_id "power:+3V3")
 		(at 148.59 58.42 270)
@@
 			)
 		)
-		(property "Footprint" "MX_Only:MXOnly-1U"
+		(property "Footprint" "MX_Only:MXOnly-1U-NoLED"
 			(at 44.45 44.45 0)
 			(hide yes)

Commit message: feat: finished preliminary wiring
Parts:
- added J4, J6: Conn_01x07, Connector_FFC-FPC:Molex_200528-0070_1x07-1MP_P1.00mm_Horizontal, symbol Connector_Generic:Conn_01x07
Connections:
- net +3V3: now also J6.2 (Pin_2)
- net COL0: now also J4.1 (Pin_1)
- net COL1: now also J4.2 (Pin_2)
- net EC1: now also J6.5 (Pin_5)
- net EC2: now also J6.7 (Pin_7)
- net GND: now also J6.4 (Pin_4), J6.6 (Pin_6)
- net ROW0: now also J4.7 (Pin_7)
- net ROW1: now also J4.6 (Pin_6)
- net ROW2: now also J4.5 (Pin_5)
- net ROW3: now also J4.4 (Pin_4)
- net ROW4: now also J4.3 (Pin_3)
- net SCL: now also J6.1 (Pin_1)
- net SDA: now also J6.3 (Pin_3)
Other:
- moved on the sheet: D1, D10, D2, D3, D4, D5, D6, D7, D8, D9, Display1, MX1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
