File: kicad/thorn_USB.kicad_sch (KiCad schematic)
At the start: 7 parts, among them J1 Conn_01x04, J2 USB_C_Receptacle_USB2.0_14P, U2 NCP1117-3.3_SOT223

Commit message: feat: finished preliminary wiring
Parts:
- removed J1: Conn_01x04, Connector_JST:JST_SH_SM04B-SRSS-TB_1x04-1MP_P1.00mm_Horizontal, symbol Connector_Generic:Conn_01x04
- J2: footprint Connector_USB:USB_C_Receptacle_HRO_TYPE-C-31-M-17 -> Connector_USB:USB_C_Receptacle_JAE_DX07S016JA1R1500
Other:
- moved on the sheet: C1, C2, J2, R1, R2, U2

Commit message: feat: change pcb to preliminary final design
Parts:
- added U4: SRV05-4, Package_TO_SOT_SMD:SOT-23-6, symbol Power_Protection:SRV05-4
Connections:
- net D+: now also U4.1 (IO1)
- net D-: now also U4.6 (IO4)
- net GND: now also U4.2 (VN)
- new net +5V: U4.5 (VP)
- no-connect marks 0 -> 2
Other:
- title: (none) -> USB Circuit
- moved on the sheet: C1, C2, J2, R1, R2, U2
